File: doc/designspec/diagrams/sens/sens.sch (KiCad schematic (older format))
At the start: 16 parts

Commit message: Schematics should be finished now, aref fixed and LCD changed to 4 mod pin, lp filters included, capacitator for AVCC aswell
Connections:
- wire segments 61 -> 62
Other:
- moved on the sheet: C?
Changed lines of the file:
@@
-$EndComp
-$Comp
-L sens-rescue:ATmega1284-PU-MCU_Microchip_ATmega U?
-U 1 1 5BDC5F4E
-P 5600 3150
-F 0 "U?" H 5600 1064 50  0000 C CNN
-F 1 "ATmega1284-PU" H 5600 973 50  0000 C CNN
-F 2 "Package_DIP:DIP-40_W15.24mm" H 5600 3150 50  0001 C CIN
-F 3 "http://ww1.microchip.com/downloads/en/DeviceDoc/Atmel-8272-8-bit-AVR-microcontroller-ATmega164A_PA-324A_PA-644A_PA-1284_P_datasheet.pdf" H 5600 3150 50  0001 C CNN
-	1    5600 3150
-	1    0    0    -1
 $EndComp
 $Comp
@@
 Wire Wire Line
 	6200 3050 6850 3050
-Wire Wire Line
-	7400 4750 7250 4750
-Wire Wire Line
-	7250 4750 7250 4250
-Wire Wire Line
-	7250 4250 6200 4250
-Wire Wire Line
-	7400 4850 7150 4850
-Wire Wire Line
-	7150 4850 7150 4350
-Wire Wire Line
-	6200 4350 7150 4350
-Wire Wire Line
-	7400 4950 7050 4950
-Wire Wire Line
-	7050 4950 7050 4450
-Wire Wire Line
-	7050 4450 6200 4450
-Wire Wire Line
-	7400 5450 6500 5450
-Wire Wire Line
-	6500 5450 6500 3950
-Wire Wire Line
-	6500 3950 6200 3950
 $Comp
 L power:+5V #PWR?
@@
 $EndComp
 Wire Wire Line
-	7400 4650 7300 4650
-Wire Wire Line
-	7300 4650 7300 4150
-Wire Wire Line
-	7300 4150 6200 4150
-Wire Wire Line
 	6200 3750 7150 3750
 Wire Wire Line
@@
 	6200 3450 7150 3450
 Wire Wire Line
-	8200 2650 6200 2650
-Wire Wire Line
 	8650 3100 8400 3100
 Wire Wire Line
@@
 Wire Wire Line
 	8400 2550 6200 2550
-Wire Wire Line
-	8650 3900 8650 3450
-Wire Wire Line
-	8650 3450 8200 3450
-Wire Wire Line
-	8200 3450 8200 2650
 $Comp
 L sens-rescue:A112X-hall-effect HALLEFFECTSENSOR?
@@
 L pspice:CAP C?
 U 1 1 5BEA46CC
-P 5650 800
-F 0 "C?" V 5335 800 50  0000 C CNN
-F 1 "CAP" V 5426 800 50  0000 C CNN
-F 2 "" H 5650 800 50  0001 C CNN
-F 3 "" H 5650 800 50  0001 C CNN
-	1    5650 800
+P 5350 800
+F 0 "C?" V 5035 800 50  0000 C CNN
+F 1 "CAP" V 5126 800 50  0000 C CNN
+F 2 "" H 5350 800 50  0001 C CNN
+F 3 "" H 5350 800 50  0001 C CNN
+	1    5350 800
 	0    1    1    0
 $EndComp
@@
 L power:GNDREF #PWR?
 U 1 1 5BEA491F
-P 5400 800
-F 0 "#PWR?" H 5400 550 50  0001 C CNN
-F 1 "GNDREF" V 5405 672 50  0000 R CNN
-F 2 "" H 5400 800 50  0001 C CNN
-F 3 "" H 5400 800 50  0001 C CNN
-	1    5400 800
-	0    1    1    0
-$EndComp
-Wire Wire Line
-	5700 1150 5900 1150
-Wire Wire Line
-	5900 1150 5900 1050
-Wire Wire Line
-	5600 1150 5600 1050
-Wire Wire Line
-	5600 1050 5900 1050
-Connection ~ 5900 1050
-Wire Wire Line
-	5900 1050 5900 800
+P 5100 800
+F 0 "#PWR?" H 5100 550 50  0001 C CNN
+F 1 "GNDREF" V 5105 672 50  0000 R CNN
+F 2 "" H 5100 800 50  0001 C CNN
+F 3 "" H 5100 800 50  0001 C CNN
+	1    5100 800
+	0    1    1    0
+$EndComp
+$Comp
+L power:+5V #PWR?
+U 1 1 5BEA6E18
+P 5600 800
+F 0 "#PWR?" H 5600 650 50  0001 C CNN
+F 1 "+5V" V 5615 928 50  0000 L CNN
+F 2 "" H 5600 800 50  0001 C CNN
+F 3 "" H 5600 800 50  0001 C CNN
+	1    5600 800
+	0    1    1    0
+$EndComp
+Wire Wire Line
+	8250 4500 8250 4250
+Wire Wire Line
+	8250 4250 6200 4250
+Wire Wire Line
+	8650 3900 8050 3900
+Wire Wire Line
+	8050 3900 8050 4350
+Wire Wire Line
+	8050 4350 6200 4350
+Wire Wire Line
+	5600 800  5600 950
+Connection ~ 5600 800
+$Comp
+L sens-rescue:ATmega1284-PU-MCU_Microchip_ATmega U?
+U 1 1 5BDC5F4E
+P 5600 3150
+F 0 "U?" H 5600 1064 50  0000 C CNN
+F 1 "ATmega1284-PU" H 5600 973 50  0000 C CNN
+F 2 "Package_DIP:DIP-40_W15.24mm" H 5600 3150 50  0001 C CIN
+F 3 "http://ww1.microchip.com/downloads/en/DeviceDoc/Atmel-8272-8-bit-AVR-microcontroller-ATmega164A_PA-324A_PA-644A_PA-1284_P_datasheet.pdf" H 5600 3150 50  0001 C CNN
+	1    5600 3150
+	1    0    0    -1
+$EndComp
+Wire Wire Line
+	5700 1150 5700 950
+Wire Wire Line
+	5700 950  5600 950
+Connection ~ 5600 950
+Wire Wire Line
+	5600 950  5600 1150
+$Comp
+L power:GNDREF #PWR?
+U 1 1 5BEC8E66
+P 8150 4450
+F 0 "#PWR?" H 8150 4200 50  0001 C CNN
+F 1 "GNDREF" V 8155 4322 50  0000 R CNN
+F 2 "" H 8150 4450 50  0001 C CNN
+F 3 "" H 8150 4450 50  0001 C CNN
+	1    8150 4450
+	0    1    1    0
+$EndComp
+Wire Wire Line
+	8150 4500 8150 4450
+Wire Wire Line
+	7400 5050 7250 5050
+Wire Wire Line
+	7250 5050 7250 4450
+Wire Wire Line
+	7250 4450 6200 4450
+Wire Wire Line
+	7400 5150 7150 5150
+Wire Wire Line
+	7150 5150 7150 4550
+Wire Wire Line
+	7150 4550 6200 4550
+Wire Wire Line
+	7400 5250 7050 5250
+Wire Wire Line
+	7050 5250 7050 4650
+Wire Wire Line
+	7050 4650 6200 4650
+Wire Wire Line
+	7400 5350 6950 5350
+Wire Wire Line
+	6950 5350 6950 4750
+Wire Wire Line
+	6950 4750 6200 4750
+Wire Wire Line
+	6800 5450 6800 4850
+Wire Wire Line
+	6800 4850 6200 4850
+Wire Wire Line
+	6800 5450 7400 5450
+$Comp
+L power:+5V #PWR?
+U 1 1 5BED369E
+P 5000 2050
+F 0 "#PWR?" H 5000 1900 50  0001 C CNN
+F 1 "+5V" V 5015 2178 50  0000 L CNN
+F 2 "" H 5000 2050 50  0001 C CNN
+F 3 "" H 5000 2050 50  0001 C CNN
+	1    5000 2050
+	0    -1   -1   0
+$EndComp
 $EndSCHEMATC

Commit message: Fixed pins on LCD in sens
Connections:
- wire segments 62 -> 74
Other:
- moved on the sheet: J?
Changed lines of the file:
@@
 L Connector:AVR-JTAG-10 J?
 U 1 1 5BDC62E7
-P 7650 3550
-F 0 "J?" H 7271 3596 50  0000 R CNN
-F 1 "AVR-JTAG-10" H 7271 3505 50  0000 R CNN
-F 2 "" V 7500 3700 50  0001 C CNN
-F 3 " ~" H 6375 3000 50  0001 C CNN
-	1    7650 3550
+P 7650 3250
+F 0 "J?" H 7271 3296 50  0000 R CNN
+F 1 "AVR-JTAG-10" H 7271 3205 50  0000 R CNN
+F 2 "" V 7500 3400 50  0001 C CNN
+F 3 " ~" H 6375 2700 50  0001 C CNN
+	1    7650 3250
 	-1   0    0    -1
 $EndComp
@@
 L power:+5V #PWR?
 U 1 1 5BE291AC
-P 7650 2950
-F 0 "#PWR?" H 7650 2800 50  0001 C CNN
-F 1 "+5V" H 7665 3123 50  0000 C CNN
-F 2 "" H 7650 2950 50  0001 C CNN
-F 3 "" H 7650 2950 50  0001 C CNN
-	1    7650 2950
+P 7650 2650
+F 0 "#PWR?" H 7650 2500 50  0001 C CNN
+F 1 "+5V" H 7665 2823 50  0000 C CNN
+F 2 "" H 7650 2650 50  0001 C CNN
+F 3 "" H 7650 2650 50  0001 C CNN
+	1    7650 2650
 	1    0    0    -1
 $EndComp
@@
 L power:+5V #PWR?
 U 1 1 5BE291DC
-P 7750 2950
-F 0 "#PWR?" H 7750 2800 50  0001 C CNN
-F 1 "+5V" H 7765 3123 50  0000 C CNN
-F 2 "" H 7750 2950 50  0001 C CNN
-F 3 "" H 7750 2950 50  0001 C CNN
-	1    7750 2950
+P 7750 2650
+F 0 "#PWR?" H 7750 2500 50  0001 C CNN
+F 1 "+5V" H 7765 2823 50  0000 C CNN
+F 2 "" H 7750 2650 50  0001 C CNN
+F 3 "" H 7750 2650 50  0001 C CNN
+	1    7750 2650
 	1    0    0    -1
 $EndComp
@@
 $EndComp
 Wire Wire Line
-	6200 3750 7150 3750
-Wire Wire Line
-	6200 3650 7150 3650
-Wire Wire Line
-	6200 3550 7150 3550
-Wire Wire Line
-	6200 3450 7150 3450
-Wire Wire Line
-	8650 3100 8400 3100
-Wire Wire Line
-	8400 3100 8400 2550
-Wire Wire Line
-	8400 2550 6200 2550
+	6200 3750 6900 3750
+Wire Wire Line
+	6200 3650 6800 3650
+Wire Wire Line
+	6200 3550 6650 3550
 $Comp
 L sens-rescue:A112X-hall-effect HALLEFFECTSENSOR?
@@
 $EndComp
 Wire Wire Line
-	8250 4500 8250 4250
-Wire Wire Line
-	8250 4250 6200 4250
-Wire Wire Line
-	8650 3900 8050 3900
-Wire Wire Line
-	8050 3900 8050 4350
-Wire Wire Line
-	8050 4350 6200 4350
-Wire Wire Line
 	5600 800  5600 950
 Connection ~ 5600 800
@@
 Wire Wire Line
 	8150 4500 8150 4450
-Wire Wire Line
-	7400 5050 7250 5050
-Wire Wire Line
-	7250 5050 7250 4450
-Wire Wire Line
-	7250 4450 6200 4450
-Wire Wire Line
-	7400 5150 7150 5150
-Wire Wire Line
-	7150 5150 7150 4550
-Wire Wire Line
-	7150 4550 6200 4550
-Wire Wire Line
-	7400 5250 7050 5250
-Wire Wire Line
-	7050 5250 7050 4650
-Wire Wire Line
-	7050 4650 6200 4650
-Wire Wire Line
-	7400 5350 6950 5350
-Wire Wire Line
-	6950 5350 6950 4750
-Wire Wire Line
-	6950 4750 6200 4750
-Wire Wire Line
-	6800 5450 6800 4850
-Wire Wire Line
-	6800 4850 6200 4850
-Wire Wire Line
-	6800 5450 7400 5450
 $Comp
 L power:+5V #PWR?
@@
 	0    -1   -1   0
 $EndComp
+Wire Wire Line
+	8100 3100 8650 3100
+Wire Wire Line
+	8650 3900 8150 3900
+Wire Wire Line
+	7400 5050 7200 5050
+Wire Wire Line
+	7200 5050 7200 4550
+Wire Wire Line
+	7200 4550 6200 4550
+Wire Wire Line
+	6200 3450 6400 3450
+Wire Wire Line
+	6400 3450 6400 3150
+Wire Wire Line
+	6400 3150 7150 3150
+Wire Wire Line
+	6650 3550 6650 3250
+Wire Wire Line
+	6650 3250 7150 3250
+Wire Wire Line
+	6800 3650 6800 3350
+Wire Wire Line
+	6800 3350 7150 3350
+Wire Wire Line
+	6900 3750 6900 3450
+Wire Wire Line
+	6900 3450 7150 3450
+Wire Wire Line
+	7400 5150 7050 5150
+Wire Wire Line
+	7050 5150 7050 4650
+Wire Wire Line
+	7050 4650 6200 4650
+Wire Wire Line
+	7400 5250 6950 5250
+Wire Wire Line
+	6950 5250 6950 4750
+Wire Wire Line
+	6950 4750 6200 4750
+Wire Wire Line
+	7400 5350 6850 5350
+Wire Wire Line
+	6850 5350 6850 4850
+Wire Wire Line
+	6850 4850 6200 4850
+Wire Wire Line
+	8150 3900 8150 4350
+Wire Wire Line
+	8150 4350 7150 4350
+Wire Wire Line
+	7150 4350 7150 4450
+Wire Wire Line
+	7150 4450 6200 4450
+Wire Wire Line
+	8100 3100 8100 4300
+Wire Wire Line
+	8100 4300 7050 4300
+Wire Wire Line
+	7050 4300 7050 4350
+Wire Wire Line
+	7050 4350 6200 4350
+Wire Wire Line
+	7400 5450 6350 5450
+Wire Wire Line
+	6350 5450 6350 4250
+Wire Wire Line
+	6350 4250 6200 4250
+Wire Wire Line
+	8250 4150 6200 4150
+Wire Wire Line
+	8250 4150 8250 4500
+$Comp
+L power:GNDREF #PWR?
+U 1 1 5BE5E3AA
+P 7650 3850
+F 0 "#PWR?" H 7650 3600 50  0001 C CNN
+F 1 "GNDREF" H 7655 3677 50  0000 C CNN
+F 2 "" H 7650 3850 50  0001 C CNN
+F 3 "" H 7650 3850 50  0001 C CNN
+	1    7650 3850
+	1    0    0    -1
+$EndComp
 $EndSCHEMATC

Commit message: fuck
Parts:
- _?: symbol jma162a:JMA162A -> sens-rescue:JMA162A-jma162a
Other:
- moved on the sheet: 100nF, 18kohm, AVSTÅNDSMÄTARE(FRAM), AVSTÅNDSMÄTARE(SIDA), C?, HALLEFFECTSENSOR?, J?, KRISTALLOSCILLATOR, R?, U?, U?A
