File: doc/designspec/diagrams/styr/styr.sch (KiCad schematic (older format))
At the start: 8 parts

Commit message: fixed styrpins to 4 mod databuss instead, adde more info about lcd in subsection styr_ctrl
Parts:
- U?: symbol styr-rescue:ATmega1284P-PU-MCU_Microchip_ATmega -> styr-rescue:ATmega1284P-PU-MCU_Microchip_ATmega-styr-rescue
- U?: symbol styr-rescue:IQEXO-3-exo3 -> styr-rescue:IQEXO-3-exo3-styr-rescue
- _?: symbol styr-rescue:JMA162A-jma162a -> styr-rescue:JMA162A-jma162a-styr-rescue
Connections:
- wire segments 57 -> 45
Other:
- note added: "4->4, 5->5, 6->6, 7->7"
- note removed: "0->0, 1->1, 2->2, 3->3, 4->4, 5->5, 6->6"
Changed lines of the file:
@@
 $EndComp
 $Comp
-L styr-rescue:ATmega1284P-PU-MCU_Microchip_ATmega U?
+L styr-rescue:ATmega1284P-PU-MCU_Microchip_ATmega-styr-rescue U?
 U 1 1 5BEA84E2
 P 2850 3150
@@
 $EndComp
 $Comp
-L styr-rescue:IQEXO-3-exo3 U?
+L styr-rescue:IQEXO-3-exo3-styr-rescue U?
 U 1 1 5BEB103D
 P 1350 2150
@@
 SS
 $Comp
-L styr-rescue:JMA162A-jma162a _?
+L styr-rescue:JMA162A-jma162a-styr-rescue _?
 U 1 1 5BEDF369
 P 6800 2300
@@
 Text Label 4150 4550 0    50   ~ 0
 PWM_MOTOR
-$Comp
-L power:GNDREF #PWR?
-U 1 1 5BE49225
-P 7050 1450
-F 0 "#PWR?" H 7050 1200 50  0001 C CNN
-F 1 "GNDREF" H 7055 1277 50  0000 C CNN
-F 2 "" H 7050 1450 50  0001 C CNN
-F 3 "" H 7050 1450 50  0001 C CNN
-	1    7050 1450
-	-1   0    0    1
-$EndComp
-Wire Wire Line
-	3550 1450 3550 1550
-Wire Wire Line
-	3550 1550 3450 1550
-Connection ~ 3550 1450
-Wire Wire Line
-	3550 1450 3450 1450
-Wire Wire Line
-	3550 1550 3550 1650
-Wire Wire Line
-	3550 1650 3450 1650
-Connection ~ 3550 1550
-Wire Wire Line
-	3550 1650 3550 1750
-Wire Wire Line
-	3550 1750 3450 1750
-Connection ~ 3550 1650
-Wire Wire Line
-	3550 1750 3550 1850
-Wire Wire Line
-	3550 1850 3450 1850
-Connection ~ 3550 1750
-Wire Wire Line
-	3550 1850 3550 1950
-Wire Wire Line
-	3550 1950 3450 1950
-Connection ~ 3550 1850
-Wire Wire Line
-	3550 1950 3550 2050
-Wire Wire Line
-	3550 2050 3450 2050
-Connection ~ 3550 1950
 Text Notes 4150 1450 0    50   ~ 0
-0->0, 1->1, 2->2, 3->3, 4->4, 5->5, 6->6
-Wire Wire Line
-	7050 1450 7050 1600
+4->4, 5->5, 6->6, 7->7
 Wire Wire Line
 	6950 1450 6950 1600
@@
 Wire Wire Line
 	6750 1450 6750 1600
-Wire Wire Line
-	6650 1450 6650 1600
-Wire Wire Line
-	6550 1450 6550 1600
-Wire Wire Line
-	6450 1450 6450 1600
-Wire Wire Line
-	6350 1450 6350 1600
-Connection ~ 6350 1450
-Wire Wire Line
-	6450 1450 6550 1450
-Connection ~ 6450 1450
-Connection ~ 6550 1450
-Wire Wire Line
-	6550 1450 6650 1450
-Wire Wire Line
-	6650 1450 6750 1450
-Connection ~ 6650 1450
-Connection ~ 6750 1450
 Wire Wire Line
 	6750 1450 6850 1450
@@
 	6850 1450 6950 1450
 Connection ~ 6850 1450
-Wire Wire Line
-	6350 1450 6450 1450
-Wire Wire Line
-	3550 1450 6350 1450
 Wire Wire Line
 	6200 2450 3450 2450
@@
 	-1   0    0    1
 $EndComp
+Wire Wire Line
+	3450 1850 3600 1850
+Wire Wire Line
+	3450 1950 3600 1950
+Wire Wire Line
+	3450 2050 3600 2050
+Wire Wire Line
+	3450 2150 3600 2150
+Wire Wire Line
+	6950 1450 7050 1450
+Wire Wire Line
+	7050 1450 7050 1600
+Connection ~ 6950 1450
+Wire Wire Line
+	6750 1450 3600 1450
+Wire Wire Line
+	3600 1450 3600 1850
+Connection ~ 6750 1450
+Connection ~ 3600 1850
+Wire Wire Line
+	3600 1850 3600 1950
+Connection ~ 3600 1950
+Wire Wire Line
+	3600 1950 3600 2050
+Connection ~ 3600 2050
+Wire Wire Line
+	3600 2050 3600 2150
+Connection ~ 7050 1450
+Connection ~ 3600 2150
 $EndSCHEMATC

Commit message: add text about representation of mission and map
Parts:
- U?: symbol styr-rescue:ATmega1284P-PU-MCU_Microchip_ATmega-styr-rescue -> styr-rescue:ATmega1284P-PU-MCU_Microchip_ATmega-styr-rescue-styr-rescue
- U?: symbol styr-rescue:IQEXO-3-exo3-styr-rescue -> styr-rescue:IQEXO-3-exo3-styr-rescue-styr-rescue
- _?: symbol styr-rescue:JMA162A-jma162a-styr-rescue -> styr-rescue:JMA162A-jma162a-styr-rescue-styr-rescue
Connections:
- wire segments 45 -> 47
Changed lines of the file:
@@
 $EndComp
 $Comp
-L styr-rescue:ATmega1284P-PU-MCU_Microchip_ATmega-styr-rescue U?
+L styr-rescue:ATmega1284P-PU-MCU_Microchip_ATmega-styr-rescue-styr-rescue U?
 U 1 1 5BEA84E2
 P 2850 3150
@@
 $EndComp
 $Comp
-L styr-rescue:IQEXO-3-exo3-styr-rescue U?
+L styr-rescue:IQEXO-3-exo3-styr-rescue-styr-rescue U?
 U 1 1 5BEB103D
 P 1350 2150
@@
 SS
 $Comp
-L styr-rescue:JMA162A-jma162a-styr-rescue _?
+L styr-rescue:JMA162A-jma162a-styr-rescue-styr-rescue _?
 U 1 1 5BEDF369
 P 6800 2300
@@
 Connection ~ 6850 1450
 Wire Wire Line
-	6200 2450 3450 2450
-Wire Wire Line
 	7150 1600 7150 1550
 Wire Wire Line
 	7150 1550 4950 1550
-Wire Wire Line
-	4950 1550 4950 2350
-Wire Wire Line
-	4950 2350 3450 2350
 $Comp
 L Device:C_Small CAP
@@
 Wire Wire Line
 	3600 2050 3600 2150
-Connection ~ 7050 1450
-Connection ~ 3600 2150
+Wire Wire Line
+	6200 2450 5700 2450
+Wire Wire Line
+	5700 2450 5700 1650
+Wire Wire Line
+	5700 1650 3450 1650
+Wire Wire Line
+	4950 1550 4950 1750
+Wire Wire Line
+	4950 1750 3450 1750
 $EndSCHEMATC

Commit message: update pin numbers lcd
Parts:
- _?: symbol styr-rescue:JMA162A-jma162a-styr-rescue-styr-rescue -> styr-rescue:JMA162A-jma162a-styr-rescue-styr-rescue-styr-rescue
Connections:
- net GNDREF: now also _?.5 (R/W); no longer _?.4 (R/W)
- net at U?.37 (PA3): now also _?.4 (RS); no longer _?.5 (RS)
Changed lines of the file:
@@
 SS
 $Comp
-L styr-rescue:JMA162A-jma162a-styr-rescue-styr-rescue _?
+L styr-rescue:JMA162A-jma162a-styr-rescue-styr-rescue-styr-rescue _?
 U 1 1 5BEDF369
 P 6800 2300
